File: Marvelou65-ergo/Hardware/Marvelou65-ergo.sch (KiCad schematic (older format))
At the start: 217 parts, among them J1 1, J2 USB_C_Receptacle_USB2.0, J3 Conn_01x04, J4 Conn_01x02, J5 Conn_01x04, J6 Conn_01x03, K1 1, M1 1, P1 1, Q1 1, Q2 AO3407, Q3 AO3407, SW1 Rotary_Encoder_Switch, SW2 SW_PUSH, SW3 SW_SPDT, SW4 SW_PUSH, T1 1, U1 1, U2 AP2112K-3.3, U3 E73-2G4M08S1C-52840, U4 USBLC6-2SC6, U5 TP4054, X1 1, Y1 1, Y2 32.768KHZ

Commit message: Add BOM file for JLC
add BOM file for fabrication
Parts:
- C10, C11, C12, C13, C14, C15, C16, C17, C2, C3, C4, C5, C6, C7, C8, C9: LCSC (none) -> C49678
- C18, C19, C20: LCSC (none) -> C15850
- D10, D11, D12, D13, D14, D15, D2, D3, D4, D5, D6, D7, D8, D9: LCSC (none) -> C114586
- D16: LCSC (none) -> C169540
- D17: LCSC (none) -> C375446
- D18: LCSC (none) -> C375450
- D19, D20, D21, D22, D23, D24, D25, D26, D27, D28, D29, D30, D31, D32, D33, D34, D35, D36, D37, D38, D39, D40, D41, D42, D43, D44, D45, D46, D48, D49, D50, D51, D52, D53, D54, D55, D56, D57, D58, D59, D60, D61, D62, D63, D64, D65, D66, D67, D68, D69, D70, D71, D72, D73, D74, D75, D76, D77, D78, D79, D80, D81, D82, D83, D84, D85, D86, D87: LCSC (none) -> C81598
- F2: LCSC (none) -> C261942
- J2: LCSC (none) -> C165948
- J4: LCSC (none) -> C157931
- Q2, Q3: LCSC (none) -> C693136
- R10: LCSC (none) -> C22975
- R11, R12, R13, R14: LCSC (none) -> C25804
- R2: LCSC (none) -> C25803
- R3: LCSC (none) -> C23252
- R4, R5: LCSC (none) -> C22976
- R6, R7: LCSC (none) -> C23186
- R8, R9: LCSC (none) -> C21190
- SW1: LCSC (none) -> C470748
- SW2, SW4: LCSC (none) -> C318884
- SW3: LCSC (none) -> C221841
- U2: LCSC (none) -> C51118
- U3: LCSC (none) -> C356849
- U4: LCSC (none) -> C558442
- U5: LCSC (none) -> C32574
- Y2: LCSC (none) -> C479190
